Commit message: added yumi model which corresponds to the model of the real yumi

File: models/robots/yumi.urdf (robot description, URDF)
Before this commit: robot yumi, 19 links, 18 joints
Joints:
- joint joint_1_l: limit lower=−2.941 upper=2.941 effort=300 velocity=3.142 -> lower=-2.941 upper=2.941 effort=300 velocity=3.142; origin xyz=0.05355 0.0725 0.41492 rpy=-0.9781 0.5716 -0.8236 -> xyz=0.05355 0.07250 0.41492 rpy=0.9781 -0.5716 2.3180
- joint joint_1_r: origin xyz=0.05355 -0.0725 0.41492 rpy=-0.9781 -0.5716 -2.3180 -> xyz=0.05355 -0.0725 0.41492 rpy=-0.9781 -0.5682 -2.3180
- joint joint_7_l: limit lower=−2.941 upper=2.941 effort=300 velocity=3.142 -> lower=-2.941 upper=2.941 effort=300 velocity=3.142
- joint joint_7_r: origin xyz=-0.03 0.17283 0 rpy=-1.571 3.142 0 -> xyz=-0.03 0.17283 0 rpy=-1.571 0 0

File: models/robots/yumi_left_arm.urdf (robot description, URDF)
Before this commit: robot yumi_left_arm, 10 links, 9 joints
Joints:
- joint joint_1_l: limit lower=−2.941 upper=2.941 effort=300 velocity=3.142 -> lower=-2.941 upper=2.941 effort=300 velocity=3.142; origin xyz=0.05355 0.0725 0.41492 rpy=-0.9781 0.5716 -0.8236 -> xyz=0.05355 0.07250 0.41492 rpy=0.9781 -0.5716 2.3180
- joint joint_7_l: limit lower=−2.941 upper=2.941 effort=300 velocity=3.142 -> lower=-2.941 upper=2.941 effort=300 velocity=3.142

File: models/robots/yumi_right_arm.urdf (robot description, URDF)
Before this commit: robot yumi_right_arm, 10 links, 9 joints
Joints:
- joint joint_1_r: origin xyz=0.05355 -0.0725 0.41492 rpy=-0.9781 -0.5716 -2.3180 -> xyz=0.05355 -0.0725 0.41492 rpy=-0.9781 -0.5682 -2.3180
- joint joint_7_r: origin xyz=-0.03 0.17283 0 rpy=-1.571 3.142 0 -> xyz=-0.03 0.17283 0 rpy=-1.571 0 0
