Commit message: modified YuMi robot not to detect autocollisions between shoulder and body + added correct inv kin to each arm (left/right)

File: models/robots/yumi_body.urdf (robot description, URDF)
Before this commit: robot yumi_body, 1 links, 0 joints
Links:
- link body: geometry collision box size=0.27 0.26 0.571; collision box size=0.3 0.26 0.17

File: models/robots/yumi_left_arm.urdf (robot description, URDF)
Before this commit: robot yumi_left_arm, 10 links, 9 joints
Links:
- link null_base: geometry collision cylinder length=0.001 radius=0.001; visual cylinder length=0.001 radius=0.001

File: models/robots/yumi_right_arm.urdf (robot description, URDF)
Before this commit: robot yumi_right_arm, 10 links, 9 joints
Links:
- link null_base: geometry collision cylinder length=0.001 radius=0.001; visual cylinder length=0.001 radius=0.001
