Commit message: fixed scale and names for kuka scene

File: models/robots/kuka_lwr.urdf (robot description, URDF)
Before this commit: robot kuka_lwr, 8 links, 7 joints
Links:
- link base: geometry collision cylinder length=0.11 radius=0.08; visual mesh filename=kukaLWR/base.wrl scale=1.0 1.0 1.0
- link link1: geometry collision cylinder length=0.2 radius=0.08; collision sphere radius=0.1
- link link2: geometry collision cylinder length=0.2 radius=0.08; visual mesh filename=kukaLWR/link2.wrl scale=1.0 1.0 1.0
- link link3: geometry collision cylinder length=0.2 radius=0.08; collision sphere radius=0.1
- link link4: geometry collision cylinder length=0.2 radius=0.08; visual mesh filename=kukaLWR/link4.wrl scale=1.0 1.0 1.0
- link link5: geometry collision cylinder length=0.13 radius=0.08; visual mesh filename=kukaLWR/link5.wrl scale=1.0 1.0 1.0
- link link6: geometry collision sphere radius=0.085; visual mesh filename=kukaLWR/link6.wrl scale=1.0 1.0 1.0
- link link7: geometry collision cylinder length=0.023 radius=0.0505; visual mesh filename=kukaLWR/link7.wrl scale=1.0 1.0 1.0

Commit message: added last link length in kuka urdf and dh models

File: models/robots/kuka_lwr.urdf (robot description, URDF)
Before this commit: robot kukaLWR, 8 links, 7 joints
Joints:
- joint joint7: origin xyz=0 0 0 rpy=-1.57079632679 0 0 -> xyz=0 0 0.078 rpy=-1.57079632679 0 0

Commit message: added last link to kuka urdf model

File: models/robots/kuka_lwr.urdf (robot description, URDF)
Before this commit: robot kukaLWR, 8 links, 7 joints
Joints:
- joint joint7: origin xyz=0 0 0.078 rpy=-1.57079632679 0 0 -> xyz=0 0.078 0 rpy=-1.57079632679 0 0
