Commit message: Allow to use (or not) the parent link with the origin.

File: kautham_models/robots/robot_descriptions/UR/ur_macro.xacro (robot description, xacro)
@@ -296,10 +296,12 @@
             </inertial>
         </link>
-        <!-- base_joint fixes base_link to the environment -->
-        <joint name="${tf_prefix}base_joint" type="fixed">
-            <xacro:insert_block name="origin" />
-            <parent link="${parent}" />
-            <child link="${tf_prefix}base_link" />
-        </joint>
+        <!-- base_joint fixes base_link to the external parent_link -->
+        <xacro:if value="${parent != ''}">
+            <joint name="${tf_prefix}base_joint" type="fixed">
+                <xacro:insert_block name="origin" />
+                <parent link="${parent}" />
+                <child link="${tf_prefix}base_link" />
+            </joint>
+        </xacro:if>
         <!-- joints - main serial chain -->
         <joint name="${tf_prefix}base_link-base_link_inertia" type="fixed">
