Commit message: Rename of the models folder. And added readmes.

File: kautham_models/robots/robot_instances/UR/ur5.urdf.xacro (robot description, xacro)
@@ -21,11 +21,15 @@
     <!--When using gazebo simulations absolute paths are necessary.-->
     <xacro:arg name="force_abs_paths" default="true" />
+    <!-- Arguments for parent and origin -->
+    <xacro:arg name="parent" default="world"/>
+    <xacro:arg name="origin_xyz" default="0 0 0"/>
+    <xacro:arg name="origin_rpy" default="0 0 0"/>
     <!-- create link fixed to the "world" -->
-    <link name="$(arg name)_base_link" />
+    <link name="$(arg parent)" />
     <!-- arm -->
     <xacro:ur_robot
         name="$(arg name)"
         tf_prefix="$(arg tf_prefix)"
-        parent="$(arg name)_base_link"
+        parent="$(arg parent)"
         joint_limits_parameters_file="$(arg joint_limit_params)"
         kinematics_parameters_file="$(arg kinematics_params)"
@@ -37,5 +41,5 @@
         force_abs_paths="$(arg force_abs_paths)"
         >
-        <origin xyz="0 0 0" rpy="0 0 0" />          <!-- position robot in the world -->
+        <origin xyz="$(arg origin_xyz)" rpy="$(arg origin_rpy)" />          <!-- position robot in the parent reference -->
     </xacro:ur_robot>
 </robot>

Commit message: Removed world link as a parent.

File: kautham_models/robots/robot_instances/UR/ur5.urdf.xacro (robot description, xacro)
@@ -22,9 +22,7 @@
     <xacro:arg name="force_abs_paths" default="true" />
     <!-- Arguments for parent and origin -->
-    <xacro:arg name="parent" default="world"/>
+    <xacro:arg name="parent" default=""/>
     <xacro:arg name="origin_xyz" default="0 0 0"/>
     <xacro:arg name="origin_rpy" default="0 0 0"/>
-    <!-- create link fixed to the "world" -->
-    <link name="$(arg parent)" />
     <!-- arm -->
     <xacro:ur_robot
@@ -41,5 +39,6 @@
         force_abs_paths="$(arg force_abs_paths)"
         >
-        <origin xyz="$(arg origin_xyz)" rpy="$(arg origin_rpy)" />          <!-- position robot in the parent reference -->
+        <!-- position robot in the parent reference -->
+        <origin xyz="$(arg origin_xyz)" rpy="$(arg origin_rpy)" />
     </xacro:ur_robot>
 </robot>
