Commit message: Removed old files and added tiago_dual_robot.

File: kautham_models/robots/robot_descriptions/tiago_robot/urdf/arm/arm.urdf.xacro (robot description, xacro)
@@ -26,6 +26,7 @@
   <xacro:property name="arm_eps" value="${0.00 if no_safety_eps else 0.07}"/>
   <!-- INCLUDES -->
-  <xacro:include filename="$(find pal_urdf_utils)/urdf/deg_to_rad.urdf.xacro" />
-  <xacro:include filename="$(find tiago_description)/urdf/arm/wrist.urdf.xacro" />
+  <!-- <xacro:include filename="$(find pal_urdf_utils)/urdf/deg_to_rad.urdf.xacro" /> -->
+  <xacro:arg name="from_tiago_arm_2_tiago_description_path" default="./../../robot_descriptions/tiago_robot"/>
+  <xacro:include filename="./wrist.urdf.xacro" />
   <!-- MACRO DEFINITION-->
   <xacro:macro name="tiago_arm" params="name parent reflect wrist_model has_ft_sensor tiago_dual *origin">
@@ -49,5 +50,5 @@
         <origin xyz="0 0 0" rpy="0 0 0" />
         <geometry>
-          <mesh filename="package://tiago_description/meshes/arm/arm_1.stl" scale="1 ${-1 * tiago_dual} ${reflect}"/>
+          <mesh filename="$(arg from_tiago_arm_2_tiago_description_path)/meshes/arm/arm_1.stl" scale="1 ${-1 * tiago_dual} ${reflect}"/>
         </geometry>
         <material name="White"/>
@@ -56,5 +57,5 @@
         <origin xyz="0 0 0" rpy="0 0 0" />
         <geometry>
-          <mesh filename="package://tiago_description/meshes/arm/arm_1_collision.dae" scale="1 ${-1 * tiago_dual} ${reflect}"/>
+          <mesh filename="$(arg from_tiago_arm_2_tiago_description_path)/meshes/arm/arm_1_collision.dae" scale="1 ${-1 * tiago_dual} ${reflect}"/>
         </geometry>
       </collision>
@@ -81,5 +82,5 @@
         <origin xyz="0 0 0" rpy="${0 * deg_to_rad} ${0 * deg_to_rad} ${0 * deg_to_rad}" />
         <geometry>
-          <mesh filename="package://tiago_description/meshes/arm/arm_2.stl" scale="1 1 ${reflect}"/>
+          <mesh filename="$(arg from_tiago_arm_2_tiago_description_path)/meshes/arm/arm_2.stl" scale="1 1 ${reflect}"/>
         </geometry>
         <material name="DarkGrey" />
@@ -89,5 +90,5 @@
         <origin xyz="0 0 0" rpy="${0 * deg_to_rad} ${0 * deg_to_rad} ${0 * deg_to_rad}" />
         <geometry>
-          <mesh filename="package://tiago_description/meshes/arm/arm_2_collision.dae" scale="1 1 ${reflect}"/>
+          <mesh filename="$(arg from_tiago_arm_2_tiago_description_path)/meshes/arm/arm_2_collision.dae" scale="1 1 ${reflect}"/>
         </geometry>
       </collision>
@@ -113,5 +114,5 @@
         <origin xyz="0 0 0" rpy="0 0 0" />
         <geometry>
-          <mesh filename="package://tiago_description/meshes/arm/arm_3.stl" scale="1 1 ${reflect}"/>
+          <mesh filename="$(arg from_tiago_arm_2_tiago_description_path)/meshes/arm/arm_3.stl" scale="1 1 ${reflect}"/>
         </geometry>
         <material name="DarkGrey" />
@@ -120,5 +121,5 @@
         <origin xyz="0 0 0" rpy="0 0 0" />
         <geometry>
-          <mesh filename="package://tiago_description/meshes/arm/arm_3_collision.dae" scale="1 1 ${reflect}"/>
+          <mesh filename="$(arg from_tiago_arm_2_tiago_description_path)/meshes/arm/arm_3_collision.dae" scale="1 1 ${reflect}"/>
         </geometry>
       </collision>
@@ -145,5 +146,5 @@
         <origin xyz="0 0 0" rpy="0 0 0" />
         <geometry>
-          <mesh filename="package://tiago_description/meshes/arm/arm_4.stl" scale="${reflect} ${reflect} ${reflect}"/>
+          <mesh filename="$(arg from_tiago_arm_2_tiago_description_path)/meshes/arm/arm_4.stl" scale="${reflect} ${reflect} ${reflect}"/>
         </geometry>
         <material name="DarkGrey" />
@@ -152,5 +153,5 @@
         <origin xyz="0 0 0" rpy="0 0 0" />
         <geometry>
-          <mesh filename="package://tiago_description/meshes/arm/arm_4_collision.dae" scale="${reflect} ${reflect} ${reflect}"/>
+          <mesh filename="$(arg from_tiago_arm_2_tiago_description_path)/meshes/arm/arm_4_collision.dae" scale="${reflect} ${reflect} ${reflect}"/>
         </geometry>
       </collision>

File: kautham_models/robots/robot_descriptions/tiago_robot/urdf/arm/wrist.urdf.xacro (robot description, xacro)
@@ -24,5 +24,6 @@
   <xacro:property name="wrist_eps" value="${0.00 if no_safety_eps else 0.02}"/>
   <!-- INCLUDES -->
-  <xacro:include filename="$(find pal_urdf_utils)/urdf/deg_to_rad.urdf.xacro" />
+  <!-- <xacro:include filename="$(find pal_urdf_utils)/urdf/deg_to_rad.urdf.xacro" /> -->
+  <xacro:arg name="from_tiago_wrist_2_tiago_description_path" default="./../../robot_descriptions/tiago_robot"/>
   <!-- MACRO DEFINITION -->
   <xacro:macro name="wrist" params="name parent wrist_model reflect">
@@ -50,5 +51,5 @@
         <origin xyz="0 0 0" rpy="0 0 0" />
         <geometry>
-          <mesh filename="package://tiago_description/meshes/arm/arm_5-${wrist_model}.stl" scale="${reflect} ${reflect} ${reflect}"/>
+          <mesh filename="$(arg from_tiago_wrist_2_tiago_description_path)/meshes/arm/arm_5-${wrist_model}.stl" scale="${reflect} ${reflect} ${reflect}"/>
         </geometry>
         <material name="LightGrey" />
@@ -57,5 +58,5 @@
         <origin xyz="0 0 0" rpy="0 0 0" />
         <geometry>
-          <mesh filename="package://tiago_description/meshes/arm/arm_5_collision-${wrist_model}.dae" scale="${reflect} ${reflect} ${reflect}"/>
+          <mesh filename="$(arg from_tiago_wrist_2_tiago_description_path)/meshes/arm/arm_5_collision-${wrist_model}.dae" scale="${reflect} ${reflect} ${reflect}"/>
         </geometry>
       </collision>
@@ -85,14 +86,14 @@
         <origin xyz="0 0 0" rpy="0 0 0" />
         <geometry>
-          <mesh filename="package://tiago_description/meshes/arm/arm_6-${wrist_model}.stl" scale="${reflect} 1 1"/>
+          <mesh filename="$(arg from_tiago_wrist_2_tiago_description_path)/meshes/arm/arm_6-${wrist_model}.stl" scale="${reflect} 1 1"/>
         </geometry>
         <material name="LightGrey" />
       </visual>
-      <collision>
+      <!-- <collision>
         <origin xyz="0 0 0" rpy="0 0 0" />
         <geometry>
-          <mesh filename="package://tiago_description/meshes/arm/arm_6_collision-${wrist_model}.dae" scale="${reflect} 1 1"/>
+          <mesh filename="$(arg from_tiago_wrist_2_tiago_description_path)/meshes/arm/arm_6_collision-${wrist_model}.dae" scale="${reflect} 1 1"/>
         </geometry>
-      </collision>
+      </collision> -->
     </link>
     <joint name="${name}_6_joint" type="revolute">

File: kautham_models/robots/robot_descriptions/tiago_robot/urdf/end_effector/end_effector.urdf.xacro (robot description, xacro)
@@ -14,18 +14,19 @@
 <robot xmlns:xacro="http://ros.org/wiki/xacro">
   <!-- INCLUDES -->
-  <xacro:include filename="$(find pal_urdf_utils)/urdf/deg_to_rad.urdf.xacro" />
-  <xacro:include filename="$(find pal_hey5_description)/urdf/pal_hey5_hand.urdf.xacro" />
+  <!-- <xacro:include filename="$(find pal_urdf_utils)/urdf/deg_to_rad.urdf.xacro" /> -->
+  <!-- <xacro:include filename="$(find pal_hey5_description)/urdf/pal_hey5_hand.urdf.xacro" /> -->
+  <xacro:arg name="pal_gripper_description_path" default="./../../robot_descriptions/pal_gripper_description"/>
   <!-- MACRO DEFINITION -->
   <xacro:macro name="tiago_end_effector" params="name parent reflect end_effector tiago_dual:=false">
     <!-- Param dependant includes -->
     <xacro:if value="${end_effector == 'pal-gripper'}">
-      <xacro:include filename="$(find pal_gripper_description)/urdf/gripper.urdf.xacro" />
+      <xacro:include filename="$(arg pal_gripper_description_path)/urdf/gripper.urdf.xacro" />
     </xacro:if>
-    <xacro:if value="${end_effector == 'robotiq-2f-85'}">
-      <xacro:include filename="$(find pal_robotiq_description)/urdf/robotiq_85_gripper.urdf.xacro" />
-    </xacro:if>
-    <xacro:if value="${end_effector == 'robotiq-2f-140'}">
-      <xacro:include filename="$(find pal_robotiq_description)/urdf/robotiq_140_gripper.urdf.xacro" />
-    </xacro:if>
+    <!-- <xacro:if value="${end_effector == 'robotiq-2f-85'}">
+      <xacro:include filename="$(arg pal_robotiq_description)/urdf/robotiq_85_gripper.urdf.xacro" />
+    </xacro:if> -->
+    <!-- <xacro:if value="${end_effector == 'robotiq-2f-140'}">
+      <xacro:include filename="$(arg pal_robotiq_description)/urdf/robotiq_140_gripper.urdf.xacro" />
+    </xacro:if> -->
     <!-- PAL Gripper -->
     <xacro:if value="${end_effector == 'pal-gripper'}">
@@ -35,17 +36,17 @@
     </xacro:if>
     <!-- Robotiq 2F-85 Gripper -->
-    <xacro:if value="${end_effector == 'robotiq-2f-85'}">
+    <!-- <xacro:if value="${end_effector == 'robotiq-2f-85'}">
       <xacro:robotiq_85_gripper prefix="${name}_" parent="${parent}">
         <origin xyz="0 0 0" rpy="${90*deg_to_rad} ${0*deg_to_rad} ${90*deg_to_rad}"/>
       </xacro:robotiq_85_gripper>
-    </xacro:if>
+    </xacro:if> -->
     <!-- Robotiq 2F-140 Gripper -->
-    <xacro:if value="${end_effector == 'robotiq-2f-140'}">
+    <!-- <xacro:if value="${end_effector == 'robotiq-2f-140'}">
       <xacro:robotiq_140_gripper prefix="${name}_" parent="${parent}">
         <origin xyz="0 0 0" rpy="${90*deg_to_rad} ${0*deg_to_rad} ${90*deg_to_rad}"/>
       </xacro:robotiq_140_gripper>
-    </xacro:if>
+    </xacro:if> -->
     <!-- Hand -->
-    <xacro:if value="${end_effector == 'pal-hey5'}">
+    <!-- <xacro:if value="${end_effector == 'pal-hey5'}">
       <xacro:pal_hey5_hand parent="${parent}" name="${name}" reflect="${reflect}">
         <origin xyz="0 0 0" rpy="0 0 0"/>
@@ -64,5 +65,5 @@
         </collision>
       </link>
-    </xacro:if>
+    </xacro:if> -->
     <!-- Custom -->
     <!--xacro:if value="${end_effector == 'custom' and not tiago_dual}">

File: kautham_models/robots/robot_descriptions/tiago_robot/urdf/head/head.urdf.xacro (robot description, xacro)
@@ -24,8 +24,9 @@
   <xacro:property name="head_eps" value="${0.00 if no_safety_eps else 0.07}" />
   <!-- INCLUDES -->
-  <xacro:include filename="$(find pal_urdf_utils)/urdf/deg_to_rad.urdf.xacro" />
-  <xacro:include filename="$(find pal_urdf_utils)/urdf/camera/xtion_pro_live.urdf.xacro" />
-  <xacro:include filename="$(find pal_urdf_utils)/urdf/camera/orbbec_astra.urdf.xacro" />
-  <xacro:include filename="$(arg eye_hand_calibration_dir)/eye_hand_calibration.urdf.xacro" />
+    <xacro:arg name="tiago_head_description_path" default="./../../robot_descriptions/tiago_robot"/>
+    <!-- <xacro:include filename="$(arg pal_urdf_utils_path)/urdf/deg_to_rad.urdf.xacro" /> -->
+  <!-- <xacro:include filename="$(arg pal_urdf_utils_path)/urdf/camera/xtion_pro_live.urdf.xacro" />
+  <xacro:include filename="$(arg pal_urdf_utils_path)/urdf/camera/orbbec_astra.urdf.xacro" />
+  <xacro:include filename="$(arg eye_hand_calibration_dir)/eye_hand_calibration.urdf.xacro" /> -->
   <!-- MACRO DEFINITION-->
   <!-- head_1 (pan) -->
@@ -40,5 +41,5 @@
         <origin xyz="0 0 0" rpy="0 0 0"/>
         <geometry>
-          <mesh filename="package://tiago_description/meshes/head/head_1.stl" scale="1 1 1"/>
+          <mesh filename="$(arg tiago_head_description_path)/meshes/head/head_1.stl" scale="1 1 1"/>
         </geometry>
         <material name="White" />
@@ -47,5 +48,5 @@
         <origin xyz="0.0 0 0" rpy="0 0 0.0" />
         <geometry>
-          <mesh filename="package://tiago_description/meshes/head/head_1_collision.dae" scale="1 1 1"/>
+          <mesh filename="$(arg tiago_head_description_path)/meshes/head/head_1_collision.dae" scale="1 1 1"/>
         </geometry>
         <material name="White" />
@@ -61,11 +62,11 @@
       <safety_controller k_position="20" k_velocity="20" soft_lower_limit="${head_1_lower_limit * deg_to_rad + head_eps}" soft_upper_limit="${head_1_upper_limit * deg_to_rad - head_eps}" />
     </joint>
-    <gazebo reference="${name}_link">
+    <!-- <gazebo reference="${name}_link">
       <mu1>0.9</mu1>
       <mu2>0.9</mu2>
-    </gazebo>
-    <gazebo reference="${name}_joint">
+    </gazebo> -->
+    <!-- <gazebo reference="${name}_joint">
       <implicitSpringDamper>1</implicitSpringDamper>
-    </gazebo>
+    </gazebo> -->
   </xacro:macro>
   <!-- head_2 (tilt) -->
@@ -80,5 +81,5 @@
         <origin xyz="0 0 0" rpy="0 0 0" />
         <geometry>
-          <mesh filename="package://tiago_description/meshes/head/head_2.stl" scale="1 1 1"/>
+          <mesh filename="$(arg tiago_head_description_path)/meshes/head/head_2.stl" scale="1 1 1"/>
         </geometry>
         <material name="White" />
@@ -87,5 +88,5 @@
         <origin xyz="0 0 0" rpy="0 0 0" />
         <geometry>
-          <mesh filename="package://tiago_description/meshes/head/head_2_collision.dae" scale="1 1 1"/>
+          <mesh filename="$(arg tiago_head_description_path)/meshes/head/head_2_collision.dae" scale="1 1 1"/>
         </geometry>
       </collision>
@@ -108,21 +109,21 @@
     <!-- Cameras-->
     <!-- Asus Xtion-->
-    <xacro:if value="${camera_model == 'asus-xtion'}">
+    <!-- <xacro:if value="${camera_model == 'asus-xtion'}">
       <xacro:xtion_pro_live name="head_front_camera" parent="${name}_2_link" camera_model="${camera_model}" camera_extrinsic_calibration_dir="${camera_extrinsic_calibration_dir}">
-        <origin xyz="${camera_position_x} ${camera_position_y} ${camera_position_z}" rpy="${camera_orientation_r} ${camera_orientation_p} ${camera_orientation_y}" />
+        <origin xyz="${camera_position_x} ${camera_position_y} ${camera_position_z}" rpy="${camera_orientation_r} ${camera_orientation_p} ${camera_orientation_y}" /> -->
         <!-- optical origin -->
-        <origin xyz="0 0 0" rpy="${-90 * deg_to_rad} ${0 * deg_to_rad} ${-90 * deg_to_rad}" />
+        <!-- <origin xyz="0 0 0" rpy="${-90 * deg_to_rad} ${0 * deg_to_rad} ${-90 * deg_to_rad}" />
       </xacro:xtion_pro_live>
-    </xacro:if>
+    </xacro:if> -->
     <!-- Orbecc Astra-->
-    <xacro:if value="${camera_model in ['orbbec-astra', 'orbbec-astra-pro']}">
+    <!-- <xacro:if value="${camera_model in ['orbbec-astra', 'orbbec-astra-pro']}">
       <xacro:orbbec_astra name="head_front_camera" parent="${name}_2_link" camera_model="${camera_model}" camera_extrinsic_calibration_dir="${camera_extrinsic_calibration_dir}">
-        <origin xyz="${camera_position_x} ${camera_position_y} ${camera_position_z}" rpy="${camera_orientation_r} ${camera_orientation_p} ${camera_orientation_y}" />
+        <origin xyz="${camera_position_x} ${camera_position_y} ${camera_position_z}" rpy="${camera_orientation_r} ${camera_orientation_p} ${camera_orientation_y}" /> -->
         <!-- optical origin -->
-        <origin xyz="0 0 0" rpy="${-90 * deg_to_rad} ${0 * deg_to_rad} ${-90 * deg_to_rad}" />
+        <!-- <origin xyz="0 0 0" rpy="${-90 * deg_to_rad} ${0 * deg_to_rad} ${-90 * deg_to_rad}" />
       </xacro:orbbec_astra>
-    </xacro:if>
+    </xacro:if> -->
     <!-- Thermal camera -->
-    <xacro:if value="${has_thermal_camera}">
+    <!-- <xacro:if value="${has_thermal_camera}">
       <joint name="thermal_camera_joint" type="fixed">
         <parent link="${head_link_name}"/>
@@ -137,5 +138,5 @@
         </inertial>
       </link>
-    </xacro:if>
+    </xacro:if> -->
   </xacro:macro>
 </robot>

File: kautham_models/robots/robot_descriptions/tiago_robot/urdf/torso/torso.urdf.xacro (robot description, xacro)
@@ -13,9 +13,10 @@
  -->
 <robot xmlns:xacro="http://ros.org/wiki/xacro">
+  <xacro:arg name="tiago_torso_description" default="./../../robot_descriptions/tiago_robot"/>
   <!-- PROPERTIES -->
   <xacro:property name="torso_max_vel" value="0.07" />
   <xacro:property name="torso_eps" value="0.02" />
   <!-- INCLUDES -->
-  <xacro:include filename="$(find pal_urdf_utils)/urdf/deg_to_rad.urdf.xacro" />
+  <xacro:include filename="$(arg pal_urdf_utils)/urdf/deg_to_rad.urdf.xacro" />
   <!-- MACRO DEFINITION-->
   <xacro:macro name="tiago_torso" params="name parent *origin">
@@ -30,5 +31,5 @@
         <origin rpy="0 0 0" xyz="0 0 0" />
         <geometry>
-          <mesh filename="package://tiago_description/meshes/torso/torso_fix.stl" scale="1 1 1"/>
+          <mesh filename="$(arg tiago_torso_description)/meshes/torso/torso_fix.stl" scale="1 1 1"/>
         </geometry>
         <material name="LightGrey"/>
@@ -67,5 +68,5 @@
         <material name="DarkGrey"/>
       </visual>
-      <collision>
+      <!-- <collision>
         <origin rpy="0 0 0" xyz="0 0 0.275" />
         <geometry>
@@ -73,5 +74,5 @@
         </geometry>
         <material name="DarkGrey"/>
-      </collision>
+      </collision> -->
     </link>
     <gazebo reference="${name}_fixed_column_link">
@@ -94,5 +95,5 @@
         <origin rpy="0 0 0" xyz="0 0 0" />
         <geometry>
-          <mesh filename="package://tiago_description/meshes/torso/torso_lift_with_arm.stl" scale="1 1 1"/>
+          <mesh filename="$(arg tiago_torso_description)/meshes/torso/torso_lift_with_arm.stl" scale="1 1 1"/>
         </geometry>
         <material name="White"/>
@@ -101,5 +102,5 @@
         <origin rpy="0 0 0" xyz="0 0 0" />
         <geometry>
-          <mesh filename="package://tiago_description/meshes/torso/torso_lift_collision_core.dae" scale="1 1 1"/>
+          <mesh filename="$(arg tiago_torso_description)/meshes/torso/torso_lift_collision_core.dae" scale="1 1 1"/>
         </geometry>
         <material name="LightGrey"/>
@@ -108,5 +109,5 @@
         <origin rpy="0 0 0" xyz="0 0 0" />
         <geometry>
-          <mesh filename="package://tiago_description/meshes/torso/torso_lift_collision_shoulder.dae" scale="1 1 1"/>
+          <mesh filename="$(arg tiago_torso_description)/meshes/torso/torso_lift_collision_shoulder.dae" scale="1 1 1"/>
         </geometry>
         <material name="LightGrey"/>
@@ -115,5 +116,5 @@
         <origin rpy="0 0 0" xyz="0 0 0" />
         <geometry>
-          <mesh filename="package://tiago_description/meshes/torso/torso_lift_collision_neck.dae" scale="1 1 1"/>
+          <mesh filename="$(arg tiago_torso_description)/meshes/torso/torso_lift_collision_neck.dae" scale="1 1 1"/>
         </geometry>
         <material name="LightGrey"/>

File: kautham_models/robots/robot_instances/tiago_robot/tiago.urdf.xacro (robot description, xacro)
@@ -23,6 +23,9 @@
 <robot xmlns:xacro="http://ros.org/wiki/xacro" name="tiago">
   <!-- ARGUMENTS -->
+  <xacro:arg name="pal_urdf_utils_path" default="./../../robot_descriptions/pal_urdf_utils"/>
+  <xacro:arg name="tiago_description" default="./../../robot_descriptions/tiago_robot"/>
   <!-- pmb2, omni_base -->
   <xacro:arg name="base_type" default="pmb2"/>
+  <xacro:arg name="base_description" default="./../../robot_descriptions/$(arg base_type)_robot"/>
   <!-- no-laser, hokuyo, sick-551, sick-561, sick-571-->
   <xacro:arg name="laser_model" default="sick-571"/>
@@ -32,9 +35,10 @@
   <xacro:arg name="arm_type" default="tiago-arm"/>
   <!-- no-ft-sensor, schunk-ft -->
-  <xacro:arg name="ft_sensor" default="schunk-ft"/>
+  <xacro:arg name="ft_sensor" default="no-ft-sensor"/>
   <!-- wrist-2010, wrist-2017 -->
   <xacro:arg name="wrist_model" default="wrist-2017"/>
+  <!-- <xacro:arg name="wrist_model" default="wrist-2010"/> -->
   <!-- no-end-effector, pal-gripper, pal-hey5, custom, robotiq-2f-85,robotiq-2f-140-->
-  <xacro:arg name="end_effector" default="pal-hey5"/>
+  <xacro:arg name="end_effector" default="pal-gripper"/>
   <!-- no-camera, orbbec-astra, orbbec-astra-pro, asus-xtion -->
   <xacro:arg name="camera_model" default="orbbec-astra"/>
@@ -106,9 +110,6 @@
   <xacro:property name="is_public_sim" value="$(arg is_public_sim)" />
   <!-- INCLUDES -->
-  <!-- Kautham paths -->
-  <xacro:arg name="tiago_description" default="./../../robot_descriptions/tiago_robot"/>
-  <xacro:arg name="base_description" default="./../../robot_descriptions/${base_type}_robot"/>
   <!-- Tools -->
-  <!-- <xacro:include filename="$(find pal_urdf_utils)/urdf/deg_to_rad.urdf.xacro" /> -->
+  <xacro:include filename="$(arg pal_urdf_utils_path)/urdf/deg_to_rad.urdf.xacro" />
   <!-- Base -->
   <xacro:include filename="$(arg base_description)/urdf/base/base_sensors.urdf.xacro" />
@@ -121,5 +122,5 @@
     <!-- FT sensor -->
     <!-- <xacro:if value="${has_ft_sensor}">
-      <xacro:include filename="$(find pal_urdf_utils)/urdf/ft_sensors/schunk.urdf.xacro" />
+      <xacro:include filename="$(arg pal_urdf_utils_path)/urdf/ft_sensors/schunk.urdf.xacro" />
     </xacro:if> -->
     <!-- End effector -->
@@ -131,7 +132,7 @@
   <xacro:include filename="$(arg tiago_description)/urdf/head/head.urdf.xacro" />
   <!-- Materials for visualization -->
-  <!-- <xacro:include filename="$(find pal_urdf_utils)/urdf/materials.urdf.xacro" /> -->
+  <xacro:include filename="$(arg pal_urdf_utils_path)/urdf/materials.urdf.xacro" />
   <!-- ROS 2 control -->
-  <xacro:include filename="$(arg tiago_description)/ros2_control/ros2_control.urdf.xacro" />
+  <!-- <xacro:include filename="$(arg tiago_description)/ros2_control/ros2_control.urdf.xacro" /> -->
   <!-- ROBOT DEFINITION -->
   <!-- Base -->
@@ -158,7 +159,7 @@
     </xacro:tiago_arm>
     <!-- FT sensor -->
-    <xacro:if value="${has_ft_sensor}">
+    <!-- <xacro:if value="${has_ft_sensor}">
       <xacro:ft_sensor name="wrist" parent="arm_tool_link" />
-    </xacro:if>
+    </xacro:if> -->
     <!-- End effector -->
     <xacro:if value="${has_end_effector}">
@@ -169,4 +170,4 @@
   <xacro:head name="head" parent="torso_lift_link"/>
   <!-- ROS 2 Control -->
-  <xacro:tiago_ros2_control />
+  <!-- <xacro:tiago_ros2_control /> -->
 </robot>
